File: kicad-designs/companion-cube-bottom/companion/companion.kicad_pcb (KiCad board)
At the start: 2 copper layers, 34 x 34 mm, 11 parts, among them J1 Conn_01x06_Male, J2 Conn_01x06_Male, J3 Conn_01x06_Male, J4 Conn_01x06_Male, J5 Conn_01x03_Female, U1 ATtiny85-20SU

Commit message: moved header
Parts:
- moved J5 4.45 mm to (19.5, 9.70)
Changed lines of the file:
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@@
   )
   (module Connector_PinHeader_2.54mm:PinHeader_1x03_P2.54mm_Vertical_SMD_Pin1Left (layer F.Cu)
-    (at 17 6 270)
+    (at 19.47 9.7 270)
     (descr "surface-mounted straight pin header, 1x03, 2.54mm pitch, single row, style 1 (pin 1 left)")
     (tags "Surface mounted pin header SMD 1x03 2.54mm single row style1 pin1 left")

Commit message: back
Parts:
- moved J5 2.47 mm to (17.0, 9.70)
Changed lines of the file:
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@@
   )
   (module Connector_PinHeader_2.54mm:PinHeader_1x03_P2.54mm_Vertical_SMD_Pin1Left (layer F.Cu)
-    (at 19.47 9.7 270)
+    (at 17 9.7 270)
     (descr "surface-mounted straight pin header, 1x03, 2.54mm pitch, single row, style 1 (pin 1 left)")
     (tags "Surface mounted pin header SMD 1x03 2.54mm single row style1 pin1 left")
